Commit message: workindg spheres for robotiq_2f_85

File: src/curobo/content/assets/robot/ur_description/ur5e_gripper.urdf (robot description, URDF)
Before this commit: robot ur5e_robot, 23 links, 22 joints
Links:
- link base_link_inertia: geometry collision mesh filename=meshes/ur5e/collision/base.stl; visual mesh filename=meshes/ur5e/visual/base.dae
- link forearm_link: geometry collision mesh filename=meshes/ur5e/collision/forearm.stl; visual mesh filename=meshes/ur5e/visual/forearm.dae
- link shoulder_link: geometry collision mesh filename=meshes/ur5e/collision/shoulder.stl; visual mesh filename=meshes/ur5e/visual/shoulder.dae
- link upper_arm_link: geometry collision mesh filename=meshes/ur5e/collision/upperarm.stl; visual mesh filename=meshes/ur5e/visual/upperarm.dae
- link wrist_1_link: geometry collision mesh filename=meshes/ur5e/collision/wrist1.stl; visual mesh filename=meshes/ur5e/visual/wrist1.dae
- link wrist_2_link: geometry collision mesh filename=meshes/ur5e/collision/wrist2.stl; visual mesh filename=meshes/ur5e/visual/wrist2.dae
- link wrist_3_link: geometry collision mesh filename=meshes/ur5e/collision/wrist3.stl; visual mesh filename=meshes/ur5e/visual/wrist3.dae
Joints:
- joint left_inner_finger_joint: mimic joint=finger_joint multiplier=-1 offset=0 -> (none)
- joint left_inner_knuckle_joint: mimic joint=finger_joint multiplier=1 offset=0 -> (none)
- joint right_inner_finger_joint: mimic joint=finger_joint multiplier=-1 offset=0 -> (none)
- joint right_inner_knuckle_joint: mimic joint=finger_joint multiplier=1 offset=0 -> (none)
- joint right_outer_knuckle_joint: mimic joint=finger_joint multiplier=1 offset=0 -> (none)
