Commit message: added gripper support

File: src/curobo/content/assets/robot/ur_description/dual_ur5e.urdf (robot description, URDF)
Before this commit: robot ur5e_robot, 22 links, 21 joints
Joints:
- joint base_fixture_j_base_link: origin xyz=-0.04999999999999999 0.0 0.0 rpy= 0 0 0 -> xyz=-0.55 0.0 0.0 rpy= 0 0 0
- joint base_fixture_j_base_link_1: origin xyz=1.05 0.015 0.0 rpy= 0 0 0 -> xyz=0.55 0.0 0.0 rpy= 0 0 0

File: src/curobo/content/assets/robot/ur_description/ur5e_robotiq_2f_140.urdf (robot description, URDF)
Before this commit: robot ur5e_robot, 23 links, 22 joints
Joints:
- joint left_inner_finger_joint: mimic joint=finger_joint multiplier=1 offset=0 -> (none)
- joint left_inner_knuckle_joint: mimic joint=finger_joint multiplier=-1 offset=0 -> (none)
- joint right_inner_finger_joint: mimic joint=finger_joint multiplier=1 offset=0 -> (none)
- joint right_inner_knuckle_joint: mimic joint=finger_joint multiplier=-1 offset=0 -> (none)
- joint right_outer_knuckle_joint: mimic joint=finger_joint multiplier=-1 offset=0 -> (none)

Commit message: it just worked

File: src/curobo/content/assets/robot/ur_description/dual_ur5e.urdf (robot description, URDF)
Before this commit: robot ur5e_robot, 22 links, 21 joints
Joints:
- joint base_fixture_j_base_link: origin xyz=-0.55 0.0 0.0 rpy= 0 0 0 -> xyz=-0.04999999999999999 0.0 0.0 rpy= 0 0 0
- joint base_fixture_j_base_link_1: child base_link_1 -> (none); origin xyz=0.55 0.0 0.0 rpy= 0 0 0 -> xyz=1.05 0.015 0.0 rpy= 0 0 0

File: src/curobo/content/assets/robot/ur_description/dual_ur5e_gripper.urdf (robot description, URDF)
Before this commit: robot ur5e_robot, 46 links, 45 joints
Joints:
- joint finger_joint: limit lower=0 upper=0.8 effort=100000 velocity=100.2 -> lower=0 upper=0.8 effort=5 velocity=100.2
- joint finger_joint_1: limit lower=0 upper=0.8 effort=100000 velocity=100.2 -> lower=0 upper=0.8 effort=5 velocity=100.2
- joint left_inner_finger_joint: limit lower=-0.8 upper=0 effort=100000 velocity=100.2 -> lower=-0.8 upper=0 effort=5 velocity=100.2; mimic (none) -> joint=finger_joint multiplier=-1 offset=0
- joint left_inner_finger_joint_1: limit lower=-0.8 upper=0 effort=100000 velocity=100.2 -> lower=-0.8 upper=0 effort=5 velocity=100.2; mimic (none) -> joint=finger_joint_1 multiplier=-1 offset=0
- joint left_inner_knuckle_joint: limit lower=0 upper=0.8 effort=100000 velocity=100.2 -> lower=0 upper=0.8 effort=5 velocity=100.2; mimic (none) -> joint=finger_joint multiplier=1 offset=0
- joint left_inner_knuckle_joint_1: limit lower=0 upper=0.8 effort=100000 velocity=100.2 -> lower=0 upper=0.8 effort=5 velocity=100.2; mimic (none) -> joint=finger_joint_1 multiplier=1 offset=0
- joint right_inner_finger_joint: limit lower=-0.8 upper=0 effort=100000 velocity=100.2 -> lower=-0.8 upper=0 effort=5 velocity=100.2; mimic (none) -> joint=finger_joint multiplier=-1 offset=0
- joint right_inner_finger_joint_1: limit lower=-0.8 upper=0 effort=100000 velocity=100.2 -> lower=-0.8 upper=0 effort=5 velocity=100.2; mimic (none) -> joint=finger_joint_1 multiplier=-1 offset=0
- joint right_inner_knuckle_joint: limit lower=0 upper=0.8 effort=100000 velocity=100.2 -> lower=0 upper=0.8 effort=5 velocity=100.2; mimic (none) -> joint=finger_joint multiplier=1 offset=0
- joint right_inner_knuckle_joint_1: limit lower=0 upper=0.8 effort=100000 velocity=100.2 -> lower=0 upper=0.8 effort=5 velocity=100.2; mimic (none) -> joint=finger_joint_1 multiplier=1 offset=0
- joint right_outer_knuckle_joint: limit lower=0 upper=0.81 effort=100000 velocity=100.2 -> lower=0 upper=0.8 effort=5 velocity=100.2; mimic (none) -> joint=finger_joint multiplier=1 offset=0
- joint right_outer_knuckle_joint_1: limit lower=0 upper=0.81 effort=100000 velocity=100.2 -> lower=0 upper=0.8 effort=5 velocity=100.2; mimic (none) -> joint=finger_joint_1 multiplier=1 offset=0
