Commit message: dual arm urdf and yml with grippers

File: src/curobo/content/assets/robot/ur_description/dual_ur5e_gripper.urdf (robot description, URDF)
Before this commit: robot ur5e_robot, 23 links, 22 joints
Links:
- added link base_fixture_link
- added link base_link_1
- added link base_link_inertia_1, mass 4.0; collision mesh filename=meshes/ur5e/collision/base.stl; visual mesh filename=meshes/ur5e/visual/base.dae
- added link flange_1
- added link forearm_link_1, mass 2.275; collision mesh filename=meshes/ur5e/collision/forearm.stl; visual mesh filename=meshes/ur5e/visual/forearm.dae
- added link shoulder_link_1, mass 3.7; collision mesh filename=meshes/ur5e/collision/shoulder.stl; visual mesh filename=meshes/ur5e/visual/shoulder.dae
- added link tool1
- added link upper_arm_link_1, mass 8.393; collision mesh filename=meshes/ur5e/collision/upperarm.stl; visual mesh filename=meshes/ur5e/visual/upperarm.dae
- added link wrist_1_link_1, mass 1.219; collision mesh filename=meshes/ur5e/collision/wrist1.stl; visual mesh filename=meshes/ur5e/visual/wrist1.dae
- added link wrist_2_link_1, mass 1.219; collision mesh filename=meshes/ur5e/collision/wrist2.stl; visual mesh filename=meshes/ur5e/visual/wrist2.dae
- added link wrist_3_link_1, mass 0.1879; collision mesh filename=meshes/ur5e/collision/wrist3.stl; visual mesh filename=meshes/ur5e/visual/wrist3.dae
Joints:
- added joint base_fixture_j_base_link: type fixed, parent base_fixture_link, child base_link, origin xyz=-0.55 0.0 0.0 rpy= 0 0 0
- added joint base_fixture_j_base_link_1: type fixed, parent base_fixture_link, child base_link_1, origin xyz=0.55 0.0 0.0 rpy= 0 0 0
- added joint base_link-base_link_inertia_1: type fixed, parent base_link_1, child base_link_inertia_1, origin xyz=0 0 0 rpy=0 0 3.141592653589793
- added joint elbow_joint_1: type revolute, parent upper_arm_link_1, child forearm_link_1, origin xyz=-0.425 0 0 rpy=0 0 0, axis 0 0 1, limit lower=-3.141592653589793 upper=3.141592653589793 effort=150.0 velocity=3.141592653589793
- added joint flange-tool1: type fixed, parent flange_1, child tool1, origin xyz=0 0 0 rpy=0 0 0
- added joint shoulder_lift_joint_1: type revolute, parent shoulder_link_1, child upper_arm_link_1, origin xyz=0 0 0 rpy=1.570796327 0 0, axis 0 0 1, limit lower=-6.283185307179586 upper=6.283185307179586 effort=150.0 velocity=3.141592653589793
- added joint shoulder_pan_joint_1: type revolute, parent base_link_inertia_1, child shoulder_link_1, origin xyz=0 0 0.1625 rpy=0 0 0, axis 0 0 1, limit lower=-6.283185307179586 upper=6.283185307179586 effort=150.0 velocity=3.141592653589793
- added joint wrist_1_joint_1: type revolute, parent forearm_link_1, child wrist_1_link_1, origin xyz=-0.3922 0 0.1333 rpy=0 0 0, axis 0 0 1, limit lower=-6.283185307179586 upper=6.283185307179586 effort=28.0 velocity=3.141592653589793
- added joint wrist_2_joint_1: type revolute, parent wrist_1_link_1, child wrist_2_link_1, origin xyz=0 -0.0997 -2.044881182297852e-11 rpy=1.570796327 0 0, axis 0 0 1, limit lower=-6.283185307179586 upper=6.283185307179586 effort=28.0 velocity=3.141592653589793
- added joint wrist_3-flange_1: type fixed, parent wrist_3_link_1, child flange_1, origin xyz=0 0 0 rpy=0 0 0
- added joint wrist_3_joint_1: type revolute, parent wrist_2_link_1, child wrist_3_link_1, origin xyz=0 0.0996 -2.042830148012698e-11 rpy=1.570796326589793 3.141592653589793 3.141592653589793, axis 0 0 1, limit lower=-6.283185307179586 upper=6.283185307179586 effort=28.0 velocity=3.141592653589793
- joint base_link-base_fixed_joint: origin xyz=0 0 0 rpy=0 0 3.14159265359 -> xyz=0 0 0 rpy=0 0 0
- joint base_link-base_link_inertia: origin xyz=0 0 0 rpy=0 0 3.14159265359 -> xyz=0 0 0 rpy=0 0 3.141592653589793
- joint elbow_joint: limit lower=-3.14159265359 upper=3.14159265359 effort=150000.0 velocity=3000.14159265359 -> lower=-3.141592653589793 upper=3.141592653589793 effort=150.0 velocity=3.141592653589793
- joint shoulder_lift_joint: limit lower=-6.25 upper=6.25 effort=150000.0 velocity=3000.14159265359 -> lower=-6.283185307179586 upper=6.283185307179586 effort=150.0 velocity=3.141592653589793
- joint shoulder_pan_joint: limit lower=-6.25 upper=6.25 effort=150000.0 velocity=3000.14159265359 -> lower=-6.283185307179586 upper=6.283185307179586 effort=150.0 velocity=3.141592653589793
- joint wrist_1_joint: limit lower=-6.25 upper=6.25 effort=28000.0 velocity=3000.14159265359 -> lower=-6.283185307179586 upper=6.283185307179586 effort=28.0 velocity=3.141592653589793
- joint wrist_2_joint: limit lower=-6.25 upper=6.25 effort=28000.0 velocity=3000.14159265359 -> lower=-6.283185307179586 upper=6.283185307179586 effort=28.0 velocity=3.141592653589793; origin xyz=0 -0.0997 -2.0448811823e-11 rpy=1.570796327 0 0 -> xyz=0 -0.0997 -2.044881182297852e-11 rpy=1.570796327 0 0
- joint wrist_3_joint: limit lower=-6.25 upper=6.25 effort=28000.0 velocity=3000.14159265359 -> lower=-6.283185307179586 upper=6.283185307179586 effort=28.0 velocity=3.141592653589793; origin xyz=0 0.0996 -2.04283014801e-11 rpy=1.57079632659 3.14159265359 3.14159265359 -> xyz=0 0.0996 -2.042830148012698e-11 rpy=1.570796326589793 3.141592653589793 3.141592653589793

File: src/curobo/content/assets/robot/ur_description/ur5e_gripper_1.urdf (robot description, URDF)
Before this commit: robot ur5e_robot, 23 links, 22 joints
Links:
- removed link base
- removed link base_link
- removed link base_link_inertia
- removed link dummy_center_indicator_link
- removed link flange
- removed link forearm_link
- removed link left_inner_finger
- removed link left_inner_finger_pad
- removed link left_inner_knuckle
- removed link left_outer_finger
- removed link left_outer_knuckle
- removed link right_inner_finger
- removed link right_inner_finger_pad
- removed link right_inner_knuckle
- removed link right_outer_finger
- removed link right_outer_knuckle
- removed link robotiq_arg2f_base_link
- removed link shoulder_link
- removed link tool0
- removed link upper_arm_link
- removed link wrist_1_link
- removed link wrist_2_link
- removed link wrist_3_link
- added link base_1
- added link base_link_1
- added link base_link_inertia_1, mass 4.0; collision mesh filename=meshes/ur5e/collision/base.stl; visual mesh filename=meshes/ur5e/visual/base.dae
- added link dummy_center_indicator_link_1
- added link flange_1
- added link forearm_link_1, mass 2.275; collision mesh filename=meshes/ur5e/collision/forearm.stl; visual mesh filename=meshes/ur5e/visual/forearm.dae
- added link left_inner_finger_1, mass 0.0104003125914103; collision mesh filename=gripper/collision/robotiq_arg2f_85_inner_finger.obj scale=0.001 0.001 0.001; visual mesh filename=gripper/visual/robotiq_arg2f_85_inner_finger.dae scale=0.001 0.001 0.001
- added link left_inner_finger_pad_1, mass 0.11; collision box size=0.022 0.015 0.07; visual box size=0.022 0.015 0.07
- added link left_inner_knuckle_1, mass 0.0271177346495152; collision mesh filename=gripper/collision/robotiq_arg2f_85_inner_knuckle.dae scale=0.001 0.001 0.001; visual mesh filename=gripper/visual/robotiq_arg2f_85_inner_knuckle.dae scale=0.001 0.001 0.001
- added link left_outer_finger_1, mass 0.022614240507152; collision mesh filename=gripper/collision/robotiq_arg2f_85_outer_finger.dae scale=0.001 0.001 0.001; visual mesh filename=gripper/visual/robotiq_arg2f_85_outer_finger.dae scale=0.001 0.001 0.001
- added link left_outer_knuckle_1, mass 0.00853198276973456; collision mesh filename=gripper/collision/robotiq_arg2f_85_outer_knuckle.dae scale=0.001 0.001 0.001; visual mesh filename=gripper/visual/robotiq_arg2f_85_outer_knuckle.dae scale=0.001 0.001 0.001
- added link right_inner_finger_1, mass 0.0104003125914103; collision mesh filename=gripper/collision/robotiq_arg2f_85_inner_finger.obj scale=0.001 0.001 0.001; visual mesh filename=gripper/visual/robotiq_arg2f_85_inner_finger.dae scale=0.001 0.001 0.001
- added link right_inner_finger_pad_1, mass 0.11; collision box size=0.022 0.015 0.07; visual box size=0.022 0.015 0.07
- added link right_inner_knuckle_1, mass 0.0271177346495152; collision mesh filename=gripper/collision/robotiq_arg2f_85_inner_knuckle.dae scale=0.001 0.001 0.001; visual mesh filename=gripper/visual/robotiq_arg2f_85_inner_knuckle.dae scale=0.001 0.001 0.001
- added link right_outer_finger_1, mass 0.022614240507152; collision mesh filename=gripper/collision/robotiq_arg2f_85_outer_finger.dae scale=0.001 0.001 0.001; visual mesh filename=gripper/visual/robotiq_arg2f_85_outer_finger.dae scale=0.001 0.001 0.001
- added link right_outer_knuckle_1, mass 0.00853198276973456; collision mesh filename=gripper/collision/robotiq_arg2f_85_outer_knuckle.dae scale=0.001 0.001 0.001; visual mesh filename=gripper/visual/robotiq_arg2f_85_outer_knuckle.dae scale=0.001 0.001 0.001
- added link robotiq_arg2f_base_link_1, mass 0.22652; visual mesh filename=gripper/visual/robotiq_arg2f_85_base_link.dae scale=0.001 0.001 0.001
- added link shoulder_link_1, mass 3.7; collision mesh filename=meshes/ur5e/collision/shoulder.stl; visual mesh filename=meshes/ur5e/visual/shoulder.dae
- added link tool0_1
- added link upper_arm_link_1, mass 8.393; collision mesh filename=meshes/ur5e/collision/upperarm.stl; visual mesh filename=meshes/ur5e/visual/upperarm.dae
- added link wrist_1_link_1, mass 1.219; collision mesh filename=meshes/ur5e/collision/wrist1.stl; visual mesh filename=meshes/ur5e/visual/wrist1.dae
- added link wrist_2_link_1, mass 1.219; collision mesh filename=meshes/ur5e/collision/wrist2.stl; visual mesh filename=meshes/ur5e/visual/wrist2.dae
- added link wrist_3_link_1, mass 0.1879; collision mesh filename=meshes/ur5e/collision/wrist3.stl; visual mesh filename=meshes/ur5e/visual/wrist3.dae
Joints:
- removed joint base_link-base_fixed_joint
- removed joint base_link-base_link_inertia
- removed joint dummy_center_fixed_joint
- removed joint elbow_joint
- removed joint finger_joint
- removed joint flange-gripper
- removed joint flange-tool0
- removed joint left_inner_finger_joint
- removed joint left_inner_finger_pad_joint
- removed joint left_inner_knuckle_joint
- removed joint left_outer_finger_joint
- removed joint right_inner_finger_joint
- removed joint right_inner_finger_pad_joint
- removed joint right_inner_knuckle_joint
- removed joint right_outer_finger_joint
- removed joint right_outer_knuckle_joint
- removed joint shoulder_lift_joint
- removed joint shoulder_pan_joint
- removed joint wrist_1_joint
- removed joint wrist_2_joint
- removed joint wrist_3-flange
- removed joint wrist_3_joint
- added joint base_link-base_fixed_joint_1: type fixed, parent base_link_1, child base_1, origin xyz=0 0 0 rpy=0 0 3.14159265359
- added joint base_link-base_link_inertia_1: type fixed, parent base_link_1, child base_link_inertia_1, origin xyz=0 0 0 rpy=0 0 3.14159265359
- added joint dummy_center_fixed_joint_1: type fixed, parent robotiq_arg2f_base_link_1, child dummy_center_indicator_link_1, origin xyz=0 0 0.1725
- added joint elbow_joint_1: type revolute, parent upper_arm_link_1, child forearm_link_1, origin xyz=-0.425 0 0 rpy=0 0 0, axis 0 0 1, limit lower=-3.14159265359 upper=3.14159265359 effort=150000.0 velocity=3000.14159265359
- added joint finger_joint_1: type revolute, parent robotiq_arg2f_base_link_1, child left_outer_knuckle_1, origin xyz=0 -0.0306011 0.054904 rpy=0 0 3.141592653589793, axis 1 0 0, limit lower=0 upper=0.8 effort=100000 velocity=100.2
- added joint flange-gripper_1: type fixed, parent flange_1, child robotiq_arg2f_base_link_1, origin xyz=0 0 0 rpy=1.57079632679 0 1.57079632679
- added joint flange-tool0_1: type fixed, parent flange_1, child tool0_1, origin xyz=0 0 0 rpy=1.57079632679 0 1.57079632679
- added joint left_inner_finger_joint_1: type revolute, parent left_outer_finger_1, child left_inner_finger_1, origin xyz=0 0.0061 0.0471 rpy=0 0 0, axis 1 0 0, limit lower=-0.8757 upper=0 effort=100000 velocity=100.2
- added joint left_inner_finger_pad_joint_1: type fixed, parent left_inner_finger_1, child left_inner_finger_pad_1, origin xyz=0 -0.0190203446692936 0.03867 rpy=0 0 0, axis 0 0 1
- added joint left_inner_knuckle_joint_1: type revolute, parent robotiq_arg2f_base_link_1, child left_inner_knuckle_1, origin xyz=0 -0.0127 0.06142 rpy=0 0 3.141592653589793, axis 1 0 0, limit lower=0 upper=0.8757 effort=100000 velocity=100.2
- added joint left_outer_finger_joint_1: type fixed, parent left_outer_knuckle_1, child left_outer_finger_1, origin xyz=0 0.0315 -0.0041 rpy=0 0 0, axis 1 0 0
- added joint right_inner_finger_joint_1: type revolute, parent right_outer_finger_1, child right_inner_finger_1, origin xyz=0 0.0061 0.0471 rpy=0 0 0, axis 1 0 0, limit lower=-0.8757 upper=0 effort=100000 velocity=100.2
- added joint right_inner_finger_pad_joint_1: type fixed, parent right_inner_finger_1, child right_inner_finger_pad_1, origin xyz=0 -0.0190203446692936 0.03867 rpy=0 0 0, axis 0 0 1
- added joint right_inner_knuckle_joint_1: type revolute, parent robotiq_arg2f_base_link_1, child right_inner_knuckle_1, origin xyz=0 0.0127 0.06142 rpy=0 0 0.0, axis 1 0 0, limit lower=0 upper=0.8757 effort=100000 velocity=100.2
- added joint right_outer_finger_joint_1: type fixed, parent right_outer_knuckle_1, child right_outer_finger_1, origin xyz=0 0.0315 -0.0041 rpy=0 0 0, axis 1 0 0
- added joint right_outer_knuckle_joint_1: type revolute, parent robotiq_arg2f_base_link_1, child right_outer_knuckle_1, origin xyz=0 0.0306011 0.054904 rpy=0 0 0, axis 1 0 0, limit lower=0 upper=0.81 effort=100000 velocity=100.2
- added joint shoulder_lift_joint_1: type revolute, parent shoulder_link_1, child upper_arm_link_1, origin xyz=0 0 0 rpy=1.570796327 0 0, axis 0 0 1, limit lower=-6.25 upper=6.25 effort=150000.0 velocity=3000.14159265359
- added joint shoulder_pan_joint_1: type revolute, parent base_link_inertia_1, child shoulder_link_1, origin xyz=0 0 0.1625 rpy=0 0 0, axis 0 0 1, limit lower=-6.25 upper=6.25 effort=150000.0 velocity=3000.14159265359
- added joint wrist_1_joint_1: type revolute, parent forearm_link_1, child wrist_1_link_1, origin xyz=-0.3922 0 0.1333 rpy=0 0 0, axis 0 0 1, limit lower=-6.25 upper=6.25 effort=28000.0 velocity=3000.14159265359
- added joint wrist_2_joint_1: type revolute, parent wrist_1_link_1, child wrist_2_link_1, origin xyz=0 -0.0997 -2.0448811823e-11 rpy=1.570796327 0 0, axis 0 0 1, limit lower=-6.25 upper=6.25 effort=28000.0 velocity=3000.14159265359
- added joint wrist_3-flange_1: type fixed, parent wrist_3_link_1, child flange_1, origin xyz=0 0 0 rpy=0 -1.57079632679 -1.57079632679
- added joint wrist_3_joint_1: type revolute, parent wrist_2_link_1, child wrist_3_link_1, origin xyz=0 0.0996 -2.04283014801e-11 rpy=1.57079632659 3.14159265359 3.14159265359, axis 0 0 1, limit lower=-6.25 upper=6.25 effort=28000.0 velocity=3000.14159265359

Commit message: dual ur5e urdf finished

File: src/curobo/content/assets/robot/ur_description/dual_ur5e_gripper.urdf (robot description, URDF)
Before this commit: robot ur5e_robot, 34 links, 33 joints
Links:
- added link dummy_center_indicator_link_1
- added link left_inner_finger_1, mass 0.0104003125914103; collision mesh filename=gripper/collision/robotiq_arg2f_85_inner_finger.obj scale=0.001 0.001 0.001; visual mesh filename=gripper/visual/robotiq_arg2f_85_inner_finger.dae scale=0.001 0.001 0.001
- added link left_inner_finger_pad_1, mass 0.11; collision box size=0.022 0.015 0.07; visual box size=0.022 0.015 0.07
- added link left_inner_knuckle_1, mass 0.0271177346495152; collision mesh filename=gripper/collision/robotiq_arg2f_85_inner_knuckle.dae scale=0.001 0.001 0.001; visual mesh filename=gripper/visual/robotiq_arg2f_85_inner_knuckle.dae scale=0.001 0.001 0.001
- added link left_outer_finger_1, mass 0.022614240507152; collision mesh filename=gripper/collision/robotiq_arg2f_85_outer_finger.dae scale=0.001 0.001 0.001; visual mesh filename=gripper/visual/robotiq_arg2f_85_outer_finger.dae scale=0.001 0.001 0.001
- added link left_outer_knuckle_1, mass 0.00853198276973456; collision mesh filename=gripper/collision/robotiq_arg2f_85_outer_knuckle.dae scale=0.001 0.001 0.001; visual mesh filename=gripper/visual/robotiq_arg2f_85_outer_knuckle.dae scale=0.001 0.001 0.001
- added link right_inner_finger_1, mass 0.0104003125914103; collision mesh filename=gripper/collision/robotiq_arg2f_85_inner_finger.obj scale=0.001 0.001 0.001; visual mesh filename=gripper/visual/robotiq_arg2f_85_inner_finger.dae scale=0.001 0.001 0.001
- added link right_inner_finger_pad_1, mass 0.11; collision box size=0.022 0.015 0.07; visual box size=0.022 0.015 0.07
- added link right_inner_knuckle_1, mass 0.0271177346495152; collision mesh filename=gripper/collision/robotiq_arg2f_85_inner_knuckle.dae scale=0.001 0.001 0.001; visual mesh filename=gripper/visual/robotiq_arg2f_85_inner_knuckle.dae scale=0.001 0.001 0.001
- added link right_outer_finger_1, mass 0.022614240507152; collision mesh filename=gripper/collision/robotiq_arg2f_85_outer_finger.dae scale=0.001 0.001 0.001; visual mesh filename=gripper/visual/robotiq_arg2f_85_outer_finger.dae scale=0.001 0.001 0.001
- added link right_outer_knuckle_1, mass 0.00853198276973456; collision mesh filename=gripper/collision/robotiq_arg2f_85_outer_knuckle.dae scale=0.001 0.001 0.001; visual mesh filename=gripper/visual/robotiq_arg2f_85_outer_knuckle.dae scale=0.001 0.001 0.001
- added link robotiq_arg2f_base_link_1, mass 0.22652; visual mesh filename=gripper/visual/robotiq_arg2f_85_base_link.dae scale=0.001 0.001 0.001
Joints:
- added joint dummy_center_fixed_joint_1: type fixed, parent robotiq_arg2f_base_link_1, child dummy_center_indicator_link_1, origin xyz=0 0 0.1725
- added joint finger_joint_1: type revolute, parent robotiq_arg2f_base_link_1, child left_outer_knuckle_1, origin xyz=0 -0.0306011 0.054904 rpy=0 0 3.141592653589793, axis 1 0 0, limit lower=0 upper=0.8 effort=100000 velocity=100.2
- added joint flange-gripper_1: type fixed, parent flange_1, child robotiq_arg2f_base_link_1, origin xyz=0 0 0 rpy=1.57079632679 0 1.57079632679
- added joint left_inner_finger_joint_1: type revolute, parent left_outer_finger_1, child left_inner_finger_1, origin xyz=0 0.0061 0.0471 rpy=0 0 0, axis 1 0 0, limit lower=-0.8757 upper=0 effort=100000 velocity=100.2
- added joint left_inner_finger_pad_joint_1: type fixed, parent left_inner_finger_1, child left_inner_finger_pad_1, origin xyz=0 -0.0190203446692936 0.03867 rpy=0 0 0, axis 0 0 1
- added joint left_inner_knuckle_joint_1: type revolute, parent robotiq_arg2f_base_link_1, child left_inner_knuckle_1, origin xyz=0 -0.0127 0.06142 rpy=0 0 3.141592653589793, axis 1 0 0, limit lower=0 upper=0.8757 effort=100000 velocity=100.2
- added joint left_outer_finger_joint_1: type fixed, parent left_outer_knuckle_1, child left_outer_finger_1, origin xyz=0 0.0315 -0.0041 rpy=0 0 0, axis 1 0 0
- added joint right_inner_finger_joint_1: type revolute, parent right_outer_finger_1, child right_inner_finger_1, origin xyz=0 0.0061 0.0471 rpy=0 0 0, axis 1 0 0, limit lower=-0.8757 upper=0 effort=100000 velocity=100.2
- added joint right_inner_finger_pad_joint_1: type fixed, parent right_inner_finger_1, child right_inner_finger_pad_1, origin xyz=0 -0.0190203446692936 0.03867 rpy=0 0 0, axis 0 0 1
- added joint right_inner_knuckle_joint_1: type revolute, parent robotiq_arg2f_base_link_1, child right_inner_knuckle_1, origin xyz=0 0.0127 0.06142 rpy=0 0 0.0, axis 1 0 0, limit lower=0 upper=0.8757 effort=100000 velocity=100.2
- added joint right_outer_finger_joint_1: type fixed, parent right_outer_knuckle_1, child right_outer_finger_1, origin xyz=0 0.0315 -0.0041 rpy=0 0 0, axis 1 0 0
- added joint right_outer_knuckle_joint_1: type revolute, parent robotiq_arg2f_base_link_1, child right_outer_knuckle_1, origin xyz=0 0.0306011 0.054904 rpy=0 0 0, axis 1 0 0, limit lower=0 upper=0.81 effort=100000 velocity=100.2
- joint flange-tool1: origin xyz=0 0 0 rpy=0 0 0 -> xyz=0 0 0 rpy=1.57079632679 0 1.57079632679
- joint wrist_3-flange_1: origin xyz=0 0 0 rpy=0 0 0 -> xyz=0 0 0 rpy=0 -1.57079632679 -1.57079632679

Commit message: joint limited changed

File: src/curobo/content/assets/robot/ur_description/dual_ur5e_gripper.urdf (robot description, URDF)
Before this commit: robot ur5e_robot, 46 links, 45 joints
Joints:
- joint left_inner_finger_joint: limit lower=-0.8757 upper=0 effort=100000 velocity=100.2 -> lower=-0.8 upper=0 effort=100000 velocity=100.2
- joint left_inner_finger_joint_1: limit lower=-0.8757 upper=0 effort=100000 velocity=100.2 -> lower=-0.8 upper=0 effort=100000 velocity=100.2
- joint left_inner_knuckle_joint: limit lower=0 upper=0.8757 effort=100000 velocity=100.2 -> lower=0 upper=0.8 effort=100000 velocity=100.2
- joint left_inner_knuckle_joint_1: limit lower=0 upper=0.8757 effort=100000 velocity=100.2 -> lower=0 upper=0.8 effort=100000 velocity=100.2
- joint right_inner_finger_joint: limit lower=-0.8757 upper=0 effort=100000 velocity=100.2 -> lower=-0.8 upper=0 effort=100000 velocity=100.2
- joint right_inner_finger_joint_1: limit lower=-0.8757 upper=0 effort=100000 velocity=100.2 -> lower=-0.8 upper=0 effort=100000 velocity=100.2
- joint right_inner_knuckle_joint: limit lower=0 upper=0.8757 effort=100000 velocity=100.2 -> lower=0 upper=0.8 effort=100000 velocity=100.2
- joint right_inner_knuckle_joint_1: limit lower=0 upper=0.8757 effort=100000 velocity=100.2 -> lower=0 upper=0.8 effort=100000 velocity=100.2

Commit message: some updates

File: src/curobo/content/assets/robot/ur_description/dual_ur5e_gripper.urdf (robot description, URDF)
Before this commit: robot ur5e_robot, 46 links, 45 joints
Joints:
- joint finger_joint: limit lower=0 upper=0.8 effort=5 velocity=100.2 -> lower=0 upper=0.8 effort=1000 velocity=100.2
- joint finger_joint_1: limit lower=0 upper=0.8 effort=5 velocity=100.2 -> lower=0 upper=0.8 effort=1000 velocity=100.2
- joint left_inner_finger_joint: limit lower=-0.8 upper=0 effort=5 velocity=100.2 -> lower=-0.8 upper=0 effort=1000 velocity=100.2
- joint left_inner_finger_joint_1: limit lower=-0.8 upper=0 effort=5 velocity=100.2 -> lower=-0.8 upper=0 effort=1000 velocity=100.2
- joint left_inner_knuckle_joint: limit lower=0 upper=0.8 effort=5 velocity=100.2 -> lower=0 upper=0.8 effort=1000 velocity=100.2
- joint left_inner_knuckle_joint_1: limit lower=0 upper=0.8 effort=5 velocity=100.2 -> lower=0 upper=0.8 effort=1000 velocity=100.2
- joint right_inner_finger_joint: limit lower=-0.8 upper=0 effort=5 velocity=100.2 -> lower=-0.8 upper=0 effort=1000 velocity=100.2
- joint right_inner_finger_joint_1: limit lower=-0.8 upper=0 effort=5 velocity=100.2 -> lower=-0.8 upper=0 effort=1000 velocity=100.2
- joint right_inner_knuckle_joint: limit lower=0 upper=0.8 effort=5 velocity=100.2 -> lower=0 upper=0.8 effort=1000 velocity=100.2
- joint right_inner_knuckle_joint_1: limit lower=0 upper=0.8 effort=5 velocity=100.2 -> lower=0 upper=0.8 effort=1000 velocity=100.2
- joint right_outer_knuckle_joint: limit lower=0 upper=0.8 effort=5 velocity=100.2 -> lower=0 upper=0.8 effort=1000 velocity=100.2
- joint right_outer_knuckle_joint_1: limit lower=0 upper=0.8 effort=5 velocity=100.2 -> lower=0 upper=0.8 effort=1000 velocity=100.2
