Commit message: some updates

File: src/curobo/content/assets/robot/ur_description/dual_ur5e_gripper.urdf (robot description, URDF)
Before this commit: robot ur5e_robot, 46 links, 45 joints
Joints:
- joint base_link-base_link_inertia_1: origin xyz=0 0 0 rpy=0 0 3.141592653589793 -> xyz=0 0 0 rpy=0 0 0
- joint shoulder_lift_joint: limit lower=-6.283185307179586 upper=6.283185307179586 effort=150.0 velocity=3.141592653589793 -> lower=-3.141592653589793 upper=3.141592653589793 effort=150.0 velocity=3.141592653589793
- joint shoulder_lift_joint_1: limit lower=-6.283185307179586 upper=6.283185307179586 effort=150.0 velocity=3.141592653589793 -> lower=-3.141592653589793 upper=3.141592653589793 effort=150.0 velocity=3.141592653589793
- joint shoulder_pan_joint: limit lower=-6.283185307179586 upper=6.283185307179586 effort=150.0 velocity=3.141592653589793 -> lower=-1.57 upper=1.57 effort=150.0 velocity=3.141592653589793
- joint shoulder_pan_joint_1: limit lower=-6.283185307179586 upper=6.283185307179586 effort=150.0 velocity=3.141592653589793 -> lower=-1.57 upper=1.57 effort=150.0 velocity=3.141592653589793
- joint wrist_1_joint: limit lower=-6.283185307179586 upper=6.283185307179586 effort=28.0 velocity=3.141592653589793 -> lower=-3.141592653589793 upper=3.141592653589793 effort=150.0 velocity=3.141592653589793
- joint wrist_1_joint_1: limit lower=-6.283185307179586 upper=6.283185307179586 effort=28.0 velocity=3.141592653589793 -> lower=-3.141592653589793 upper=3.141592653589793 effort=150.0 velocity=3.141592653589793
- joint wrist_2_joint: limit lower=-6.283185307179586 upper=6.283185307179586 effort=28.0 velocity=3.141592653589793 -> lower=-3.141592653589793 upper=3.141592653589793 effort=150.0 velocity=3.141592653589793
- joint wrist_2_joint_1: limit lower=-6.283185307179586 upper=6.283185307179586 effort=28.0 velocity=3.141592653589793 -> lower=-3.141592653589793 upper=3.141592653589793 effort=150.0 velocity=3.141592653589793
- joint wrist_3_joint: limit lower=-6.283185307179586 upper=6.283185307179586 effort=28.0 velocity=3.141592653589793 -> lower=-3.141592653589793 upper=3.141592653589793 effort=150.0 velocity=3.141592653589793
- joint wrist_3_joint_1: limit lower=-6.283185307179586 upper=6.283185307179586 effort=28.0 velocity=3.141592653589793 -> lower=-3.141592653589793 upper=3.141592653589793 effort=150.0 velocity=3.141592653589793

Commit message: new weight

File: src/curobo/content/assets/robot/ur_description/dual_ur5e_gripper.urdf (robot description, URDF)
Before this commit: robot ur5e_robot, 46 links, 45 joints
Joints:
- joint elbow_joint: limit lower=-3.141592653589793 upper=3.141592653589793 effort=150.0 velocity=3.141592653589793 -> lower=0 upper=3.141592653589793 effort=150.0 velocity=3.141592653589793
- joint elbow_joint_1: limit lower=-3.141592653589793 upper=3.141592653589793 effort=150.0 velocity=3.141592653589793 -> lower=0 upper=3.141592653589793 effort=150.0 velocity=3.141592653589793
- joint wrist_1_joint: limit lower=-3.141592653589793 upper=3.141592653589793 effort=150.0 velocity=3.141592653589793 -> lower=-6.283185307179586 upper=6.283185307179586 effort=28.0 velocity=3.141592653589793
- joint wrist_1_joint_1: limit lower=-3.141592653589793 upper=3.141592653589793 effort=150.0 velocity=3.141592653589793 -> lower=-6.283185307179586 upper=6.283185307179586 effort=150.0 velocity=3.141592653589793
- joint wrist_2_joint: limit lower=-3.141592653589793 upper=3.141592653589793 effort=150.0 velocity=3.141592653589793 -> lower=-6.283185307179586 upper=6.283185307179586 effort=150.0 velocity=3.141592653589793
- joint wrist_2_joint_1: limit lower=-3.141592653589793 upper=3.141592653589793 effort=150.0 velocity=3.141592653589793 -> lower=-6.283185307179586 upper=6.283185307179586 effort=150.0 velocity=3.141592653589793
- joint wrist_3_joint: limit lower=-3.141592653589793 upper=3.141592653589793 effort=150.0 velocity=3.141592653589793 -> lower=-6.283185307179586 upper=6.283185307179586 effort=150.0 velocity=3.141592653589793
- joint wrist_3_joint_1: limit lower=-3.141592653589793 upper=3.141592653589793 effort=150.0 velocity=3.141592653589793 -> lower=-6.283185307179586 upper=6.283185307179586 effort=150.0 velocity=3.141592653589793

Commit message: new weight

File: src/curobo/content/assets/robot/ur_description/dual_ur5e_gripper.urdf (robot description, URDF)
Before this commit: robot ur5e_robot, 46 links, 45 joints
Joints:
- joint wrist_1_joint: limit lower=-6.283185307179586 upper=6.283185307179586 effort=28.0 velocity=3.141592653589793 -> lower=-3.141592653589793 upper=0 effort=150.0 velocity=3.141592653589793
- joint wrist_1_joint_1: limit lower=-6.283185307179586 upper=6.283185307179586 effort=150.0 velocity=3.141592653589793 -> lower=-3.141592653589793 upper=0 effort=150.0 velocity=3.141592653589793
- joint wrist_2_joint: limit lower=-6.283185307179586 upper=6.283185307179586 effort=150.0 velocity=3.141592653589793 -> lower=-3.141592653589793 upper=3.141592653589793 effort=150.0 velocity=3.141592653589793
- joint wrist_2_joint_1: limit lower=-6.283185307179586 upper=6.283185307179586 effort=150.0 velocity=3.141592653589793 -> lower=-3.141592653589793 upper=3.141592653589793 effort=150.0 velocity=3.141592653589793
- joint wrist_3_joint: limit lower=-6.283185307179586 upper=6.283185307179586 effort=150.0 velocity=3.141592653589793 -> lower=-3.141592653589793 upper=3.141592653589793 effort=150.0 velocity=3.141592653589793
- joint wrist_3_joint_1: limit lower=-6.283185307179586 upper=6.283185307179586 effort=150.0 velocity=3.141592653589793 -> lower=-3.141592653589793 upper=3.141592653589793 effort=150.0 velocity=3.141592653589793

Commit message: correct finger pad size and dummy tcp

File: src/curobo/content/assets/robot/ur_description/dual_ur5e_gripper.urdf (robot description, URDF)
Before this commit: robot ur5e_robot, 46 links, 45 joints
Links:
- link left_inner_finger_pad: geometry collision box size=0.022 0.015 0.05; visual box size=0.022 0.015 0.05
- link left_inner_finger_pad_1: geometry collision box size=0.022 0.015 0.05; visual box size=0.022 0.015 0.05
- link right_inner_finger_pad: geometry collision box size=0.022 0.015 0.05; visual box size=0.022 0.015 0.05
- link right_inner_finger_pad_1: geometry collision box size=0.022 0.015 0.05; visual box size=0.022 0.015 0.05
Joints:
- joint base_fixture_j_base_link: origin xyz=-0.55 0.0 0.0 rpy= 0 0 0 -> xyz=-0.55 -0.018056 0.0 rpy= 0 0 0
- joint base_fixture_j_base_link_1: origin xyz=0.55 0.0 0.0 rpy= 0 0 0 -> xyz=0.5476302 0.0 0.0 rpy= 0 0 0
- joint dummy_center_fixed_joint: origin xyz=0 0 0.1725 -> xyz=0 0 0.188
- joint dummy_center_fixed_joint_1: origin xyz=0 0 0.1725 -> xyz=0 0 0.188

Commit message: attached_object

File: src/curobo/content/assets/robot/ur_description/dual_ur5e_gripper.urdf (robot description, URDF)
Before this commit: robot ur5e_robot, 46 links, 45 joints
Links:
- removed link left_inner_finger_pad
- added link left_inner_ finger_pad, mass 0.11; collision box size=0.022 0.015 0.05; visual box size=0.022 0.015 0.05

Commit message: new calibration

File: src/curobo/content/assets/robot/ur_description/dual_ur5e_gripper.urdf (robot description, URDF)
Before this commit: robot ur5e_robot, 46 links, 45 joints
Links:
- added link left_inner_finger_pad, mass 0.11; collision box size=0.022 0.015 0.05; visual box size=0.022 0.015 0.05
Joints:
- joint base_fixture_j_base_link: origin xyz=-0.55 -0.018056 0.0 rpy= 0 0 0 -> xyz=-0.55 0 0.0 rpy=0 0 0
- joint base_fixture_j_base_link_1: origin xyz=0.5476302 0.0 0.0 rpy= 0 0 0 -> xyz=0.5496187399999999 0.02588207 0.0 rpy= 0 0 -3.105345355171964
- joint base_link-base_link_inertia_1: origin xyz=0 0 0 rpy=0 0 0 -> xyz=0 0 0 rpy=0 0 3.141592653589793
- joint dummy_center_fixed_joint: origin xyz=0 0 0.188 -> xyz=0 0 0.178
- joint dummy_center_fixed_joint_1: origin xyz=0 0 0.188 -> xyz=0 0 0.178

Commit message: fixed urdf

File: src/curobo/content/assets/robot/ur_description/dual_ur5e_gripper.urdf (robot description, URDF)
Before this commit: robot ur5e_robot, 47 links, 45 joints
Links:
- removed link left_inner_ finger_pad
